Commit message: Re-spec steering to 28 deg and align every turning-radius constant
The vehicle's real maximum steering angle is 28 deg, not the 31.5 deg the
model was built around.  In simulation the URDF *is* the vehicle, so the
old setup was internally consistent (0.58/tan(0.55) = 0.9460, exactly the
configured minimum_turning_radius) -- this change re-specs the simulated
car to the real limit and moves every dependent constant with it, so no
stale value can leak a path the car cannot physically drive.

  wheel_base 0.58 / tan(0.4887) = 1.0908 m  ->  configured 1.10

  turtle_car.urdf.xacro   steering_limit 0.55 -> 0.4887.  Both steering
                          joint limits and the Ackermann plugin read this
                          one property; verified in the expanded URDF
                          (limit lower=-0.4887 upper=0.4887,
                          <steering_limit>0.4887</steering_limit>).
  nav2_params.yaml        minimum_turning_radius 0.946 -> 1.10 for both
                          GridBased (entry, REEDS_SHEPP) and ForwardExit
                          (exit, DUBIN); regulated_linear_scaling_min_radius
                          0.946 -> 1.10 for both RPP controllers.
  t_parking_auto.yaml     minimum_turning_radius 0.946 -> 1.10
  parallel_parking_auto.yaml   same.
  auto_t_parking.py / auto_parallel_parking.py   parameter defaults and
                          the comments that quoted the old radius.

The nodes' curvature check is curvature_tolerance_factor / radius, so it
follows automatically: the accepted limit tightens from 1.2685 to 1.0909
1/m.  No literal 0.946 remains anywhere (grep-verified).

Measured effect on the parallel entry plan: max_curvature dropped from
1.057 to 0.909 1/m, i.e. exactly 1/1.10, so Smac now plans at the new
limit.  The published path was measured in the odom frame and needs none
of the extra path guards that were considered alongside this change: it
spans x[11.72, 13.26] y[2.32, 4.92], ends at (13.26, 2.32) yaw 1.609
which is inside slot_2 and 0.038 rad off the slot axis, has zero samples
outside the drivable band, and does not run out past the lane corner.

Known remaining issue, unchanged by this commit: the parallel entry
FollowPath still stalls mid-reverse ("Failed to make progress").  The
lane-edge paint was ruled out as a physical obstruction -- none of the
painted models carry collision geometry.

Co-Authored-By: Claude Sonnet 5 <noreply@anthropic.com>

File: src/t_parking_sim/urdf/turtle_car.urdf.xacro (robot description, xacro)
@@ -12,5 +12,9 @@
   <xacro:property name="wheel_radius" value="0.095"/>
   <xacro:property name="wheel_width" value="0.055"/>
-  <xacro:property name="steering_limit" value="0.55"/>
+  <!-- Real vehicle maximum steering angle: 28 deg.  The Ackermann plugin
+       and both steering joint limits read this one property, and nav2's
+       minimum_turning_radius must match wheel_base/tan(steering_limit)
+       = 0.58/tan(0.4887) = 1.091 m (configured as 1.10 for margin). -->
+  <xacro:property name="steering_limit" value="0.4887"/>
   <xacro:property name="steering_link_radius" value="0.020"/>
   <xacro:property name="steering_link_height" value="0.040"/>
