Commit message: Prepare public ROS 2 parking project

File: src/t_parking_sim/urdf/turtle_car.gazebo.xacro (robot description, xacro)
@@ -81,8 +81,8 @@
         <scan>
           <horizontal>
-            <samples>1080</samples>
-            <resolution>1</resolution>
-            <min_angle>-2.35619</min_angle>
-            <max_angle>2.35619</max_angle>
+            <samples>1440</samples>
+            <resolution>1</resolution>
+            <min_angle>${-pi}</min_angle>
+            <max_angle>${pi}</max_angle>
           </horizontal>
           <vertical>
@@ -120,8 +120,8 @@
         <scan>
           <horizontal>
-            <samples>1080</samples>
-            <resolution>1</resolution>
-            <min_angle>-2.35619</min_angle>
-            <max_angle>2.35619</max_angle>
+            <samples>1440</samples>
+            <resolution>1</resolution>
+            <min_angle>${-pi}</min_angle>
+            <max_angle>${pi}</max_angle>
           </horizontal>
           <vertical>
@@ -169,9 +169,28 @@
       <max_acceleration>1.5</max_acceleration>
       <topic>/cmd_vel</topic>
-      <odom_topic>/odom</odom_topic>
-      <tf_topic>/tf</tf_topic>
+      <!--
+        AckermannSteering integrates commanded wheel motion, so its odometry
+        continues through a physical collision.  Keep it available only as an
+        unbridged diagnostic source; it must not own ROS /odom or /tf.
+      -->
+      <odom_topic>/wheel_odom</odom_topic>
+      <tf_topic>/wheel_tf</tf_topic>
       <frame_id>odom</frame_id>
       <child_frame_id>base_footprint</child_frame_id>
       <steer_p_gain>10</steer_p_gain>
+    </plugin>
+    <!--
+      Ground-truth model odometry reads Gazebo's world pose component, including
+      collision response.  gazebo_pose_odom.py converts this absolute pose into
+      the spawn-relative odom frame used throughout the project.
+    -->
+    <plugin filename="gz-sim-odometry-publisher-system"
+            name="gz::sim::systems::OdometryPublisher">
+      <odom_frame>world</odom_frame>
+      <robot_base_frame>turtle_car</robot_base_frame>
+      <dimensions>2</dimensions>
+      <odom_publish_frequency>50</odom_publish_frequency>
+      <odom_topic>/gazebo_ground_truth/odom_absolute</odom_topic>
+      <tf_topic>/gazebo_ground_truth/tf_absolute</tf_topic>
     </plugin>
     <plugin filename="gz-sim-joint-state-publisher-system"

File: src/t_parking_sim/urdf/turtle_car.urdf.xacro (robot description, xacro)
@@ -1,26 +1,34 @@
 <?xml version="1.0"?>
 <robot xmlns:xacro="http://www.ros.org/wiki/xacro" name="turtle_car">
+  <xacro:arg name="lidar_ground_height" default="0.52"/>
   <!-- Vehicle dimensions (metres unless noted otherwise). -->
-  <xacro:property name="vehicle_length" value="0.90"/>
-  <xacro:property name="vehicle_width" value="0.45"/>
-  <xacro:property name="body_length" value="0.75"/>
-  <xacro:property name="body_width" value="0.38"/>
-  <xacro:property name="body_height" value="0.15"/>
-  <xacro:property name="wheel_base" value="0.58"/>
-  <xacro:property name="wheel_track" value="0.38"/>
-  <xacro:property name="kingpin_width" value="0.32"/>
-  <xacro:property name="wheel_radius" value="0.095"/>
-  <xacro:property name="wheel_width" value="0.055"/>
-  <!-- Real vehicle maximum steering angle: 28 deg.  The Ackermann plugin
-       and both steering joint limits read this one property, and nav2's
-       minimum_turning_radius must match wheel_base/tan(steering_limit)
-       = 0.58/tan(0.4887) = 1.091 m (configured as 1.10 for margin). -->
-  <xacro:property name="steering_limit" value="0.4887"/>
+  <xacro:property name="vehicle_length" value="1.33"/>
+  <xacro:property name="vehicle_width" value="0.78"/>
+  <xacro:property name="body_length" value="1.33"/>
+  <xacro:property name="body_width" value="0.74"/>
+  <xacro:property name="body_height" value="0.70"/>
+  <xacro:property name="body_bottom_from_ground" value="0.20"/>
+  <xacro:property name="body_center_x" value="0.020"/>
+  <xacro:property name="wheel_base" value="0.77"/>
+  <xacro:property name="wheel_track" value="0.67"/>
+  <!-- No separate kingpin measurement was supplied.  Place each steering
+       pivot at its wheel centre so the measured 0.67 m track is exact. -->
+  <xacro:property name="kingpin_width" value="${wheel_track}"/>
+  <xacro:property name="front_axle_x" value="0.385"/>
+  <xacro:property name="rear_axle_x" value="-0.385"/>
+  <xacro:property name="wheel_radius" value="0.14"/>
+  <xacro:property name="wheel_width" value="0.11"/>
+  <!-- Shared MCU/Gazebo maximum steering angle: exactly 27 deg. -->
+  <xacro:property name="steering_limit" value="0.471238898"/>
   <xacro:property name="steering_link_radius" value="0.020"/>
   <xacro:property name="steering_link_height" value="0.040"/>
-  <!-- Ahead of the front tyre envelope (x=0.385), inside the x=0.450 bumper. -->
-  <xacro:property name="laser_x" value="0.40"/>
-  <xacro:property name="laser_z_from_ground" value="0.065"/>
-  <xacro:property name="laser_radius" value="0.025"/>
+  <!-- base_link is the axle midpoint, 0.020 m behind the physical geometric
+       centre.  These offsets therefore reproduce the measured physical
+       LiDAR centres at +0.7025/-0.7025 m about the geometric centre. -->
+  <xacro:property name="front_laser_x" value="0.7225"/>
+  <xacro:property name="rear_laser_x" value="-0.6825"/>
+  <xacro:property name="laser_z_from_ground"
+                  value="${float(xacro.arg('lidar_ground_height'))}"/>
+  <xacro:property name="laser_radius" value="0.0375"/>
   <xacro:property name="laser_height" value="0.040"/>
   <!-- Total model mass is approximately 21.05 kg. -->
@@ -143,6 +151,8 @@
     <parent link="base_link"/>
     <child link="chassis_link"/>
-    <!-- Body bottom is at the wheel axle height, safely above the ground. -->
-    <origin xyz="0 0 ${body_height / 2.0}" rpy="0 0 0"/>
+    <!-- Measured body envelope: x is the physical geometric centre; z spans
+         exactly 0.20..0.90 m above ground. -->
+    <origin xyz="${body_center_x} 0 ${body_bottom_from_ground + body_height / 2.0 - wheel_radius}"
+            rpy="0 0 0"/>
   </joint>
   <xacro:steering_link name="front_left_steering_link"/>
@@ -151,5 +161,5 @@
     <parent link="base_link"/>
     <child link="front_left_steering_link"/>
-    <origin xyz="${wheel_base / 2.0} ${kingpin_width / 2.0} 0" rpy="0 0 0"/>
+    <origin xyz="${front_axle_x} ${kingpin_width / 2.0} 0" rpy="0 0 0"/>
     <axis xyz="0 0 1"/>
     <limit lower="${-steering_limit}" upper="${steering_limit}"
@@ -160,5 +170,5 @@
     <parent link="base_link"/>
     <child link="front_right_steering_link"/>
-    <origin xyz="${wheel_base / 2.0} ${-kingpin_width / 2.0} 0" rpy="0 0 0"/>
+    <origin xyz="${front_axle_x} ${-kingpin_width / 2.0} 0" rpy="0 0 0"/>
     <axis xyz="0 0 1"/>
     <limit lower="${-steering_limit}" upper="${steering_limit}"
@@ -170,5 +180,5 @@
   <xacro:wheel_link name="rear_left_wheel_link"/>
   <xacro:wheel_link name="rear_right_wheel_link"/>
-  <!-- Offset the front wheel centres from the 0.32 m kingpins to a 0.38 m track. -->
+  <!-- Front steering pivots and wheel centres share the measured track. -->
   <joint name="front_left_wheel_joint" type="continuous">
     <parent link="front_left_steering_link"/>
@@ -190,5 +200,5 @@
     <parent link="base_link"/>
     <child link="rear_left_wheel_link"/>
-    <origin xyz="${-wheel_base / 2.0} ${wheel_track / 2.0} 0" rpy="0 0 0"/>
+    <origin xyz="${rear_axle_x} ${wheel_track / 2.0} 0" rpy="0 0 0"/>
     <axis xyz="0 1 0"/>
     <limit effort="50" velocity="30"/>
@@ -198,5 +208,5 @@
     <parent link="base_link"/>
     <child link="rear_right_wheel_link"/>
-    <origin xyz="${-wheel_base / 2.0} ${-wheel_track / 2.0} 0" rpy="0 0 0"/>
+    <origin xyz="${rear_axle_x} ${-wheel_track / 2.0} 0" rpy="0 0 0"/>
     <axis xyz="0 1 0"/>
     <limit effort="50" velocity="30"/>
@@ -219,7 +229,8 @@
     <parent link="base_link"/>
     <child link="laser_link"/>
-    <origin xyz="${laser_x} 0 ${laser_z_from_ground - wheel_radius}" rpy="0 0 0"/>
-  </joint>
-  <!-- Exact centre-symmetric counterpart of the front lidar. -->
+    <origin xyz="${front_laser_x} 0 ${laser_z_from_ground - wheel_radius}" rpy="0 0 0"/>
+  </joint>
+  <!-- Rear sensor is physically symmetric about the vehicle geometric centre,
+       which is intentionally not the base_link origin. -->
   <link name="rear_laser_link">
     <inertial>
@@ -238,5 +249,5 @@
     <parent link="base_link"/>
     <child link="rear_laser_link"/>
-    <origin xyz="${-laser_x} 0 ${laser_z_from_ground - wheel_radius}"
+    <origin xyz="${rear_laser_x} 0 ${laser_z_from_ground - wheel_radius}"
             rpy="0 0 ${pi}"/>
   </joint>

Commit message: Prepare T-parking real vehicle test

File: src/t_parking_sim/urdf/turtle_car.gazebo.xacro (robot description, xacro)
@@ -2,7 +2,9 @@
 <robot xmlns:xacro="http://www.ros.org/wiki/xacro">
   <!-- Keep these joints in Gazebo's SDF conversion so the sensor frame survives. -->
-  <gazebo reference="base_footprint_joint">
-    <preserveFixedJoint>true</preserveFixedJoint>
-  </gazebo>
+  <xacro:if value="$(arg use_base_footprint)">
+    <gazebo reference="base_footprint_joint">
+      <preserveFixedJoint>true</preserveFixedJoint>
+    </gazebo>
+  </xacro:if>
   <gazebo reference="chassis_joint">
     <preserveFixedJoint>true</preserveFixedJoint>
@@ -158,5 +160,5 @@
       <left_steering_joint>front_left_steering_joint</left_steering_joint>
       <right_steering_joint>front_right_steering_joint</right_steering_joint>
-      <wheel_separation>${wheel_track}</wheel_separation>
+      <wheel_separation>${rear_wheel_track}</wheel_separation>
       <kingpin_width>${kingpin_width}</kingpin_width>
       <wheel_base>${wheel_base}</wheel_base>

File: src/t_parking_sim/urdf/turtle_car.urdf.xacro (robot description, xacro)
@@ -1,5 +1,8 @@
 <?xml version="1.0"?>
 <robot xmlns:xacro="http://www.ros.org/wiki/xacro" name="turtle_car">
-  <xacro:arg name="lidar_ground_height" default="0.52"/>
+  <xacro:arg name="include_gazebo" default="true"/>
+  <xacro:arg name="use_base_footprint" default="true"/>
+  <xacro:arg name="front_laser_z_from_base" default="-0.030"/>
+  <xacro:arg name="rear_laser_z_from_base" default="0.020"/>
   <!-- Vehicle dimensions (metres unless noted otherwise). -->
   <xacro:property name="vehicle_length" value="1.33"/>
@@ -10,24 +13,27 @@
   <xacro:property name="body_bottom_from_ground" value="0.20"/>
   <xacro:property name="body_center_x" value="0.020"/>
-  <xacro:property name="wheel_base" value="0.77"/>
-  <xacro:property name="wheel_track" value="0.67"/>
-  <!-- No separate kingpin measurement was supplied.  Place each steering
-       pivot at its wheel centre so the measured 0.67 m track is exact. -->
-  <xacro:property name="kingpin_width" value="${wheel_track}"/>
-  <xacro:property name="front_axle_x" value="0.385"/>
-  <xacro:property name="rear_axle_x" value="-0.385"/>
-  <xacro:property name="wheel_radius" value="0.14"/>
+  <xacro:property name="wheel_base" value="0.730"/>
+  <xacro:property name="front_wheel_track" value="0.775"/>
+  <xacro:property name="rear_wheel_track" value="0.785"/>
+  <!-- No separate kingpin measurement was supplied. Place each steering
+       pivot at its front wheel centre. -->
+  <xacro:property name="kingpin_width" value="${front_wheel_track}"/>
+  <xacro:property name="front_axle_x" value="0.365"/>
+  <xacro:property name="rear_axle_x" value="-0.365"/>
+  <xacro:property name="wheel_radius" value="0.135"/>
   <xacro:property name="wheel_width" value="0.11"/>
-  <!-- Shared MCU/Gazebo maximum steering angle: exactly 27 deg. -->
-  <xacro:property name="steering_limit" value="0.471238898"/>
+  <!-- Measured physical steering travel: exactly +/-22 deg. -->
+  <xacro:property name="steering_limit" value="0.383972435"/>
   <xacro:property name="steering_link_radius" value="0.020"/>
   <xacro:property name="steering_link_height" value="0.040"/>
-  <!-- base_link is the axle midpoint, 0.020 m behind the physical geometric
-       centre.  These offsets therefore reproduce the measured physical
-       LiDAR centres at +0.7025/-0.7025 m about the geometric centre. -->
-  <xacro:property name="front_laser_x" value="0.7225"/>
-  <xacro:property name="rear_laser_x" value="-0.6825"/>
-  <xacro:property name="laser_z_from_ground"
-                  value="${float(xacro.arg('lidar_ground_height'))}"/>
+  <!-- Directly measured base_link -> LiDAR transforms. base_link is at the
+       wheel centre height (0.135 m above ground); do not add that height a
+       second time to these relative z offsets. -->
+  <xacro:property name="front_laser_x" value="0.730"/>
+  <xacro:property name="front_laser_z"
+                  value="${float(xacro.arg('front_laser_z_from_base'))}"/>
+  <xacro:property name="rear_laser_x" value="-0.680"/>
+  <xacro:property name="rear_laser_z"
+                  value="${float(xacro.arg('rear_laser_z_from_base'))}"/>
   <xacro:property name="laser_radius" value="0.0375"/>
   <xacro:property name="laser_height" value="0.040"/>
@@ -106,5 +112,6 @@
   </xacro:macro>
   <!-- Root at the tyre/ground contact plane. -->
-  <link name="base_footprint">
+  <xacro:if value="$(arg use_base_footprint)">
+    <link name="base_footprint">
     <!--
       Gazebo's URDF-to-SDF converter requires an inertial block when this
@@ -116,5 +123,6 @@
                iyy="0.0001" iyz="0" izz="0.0001"/>
     </inertial>
-  </link>
+    </link>
+  </xacro:if>
   <link name="base_link">
     <inertial>
@@ -124,9 +132,11 @@
     </inertial>
   </link>
-  <joint name="base_footprint_joint" type="fixed">
-    <parent link="base_footprint"/>
-    <child link="base_link"/>
-    <origin xyz="0 0 ${wheel_radius}" rpy="0 0 0"/>
-  </joint>
+  <xacro:if value="$(arg use_base_footprint)">
+    <joint name="base_footprint_joint" type="fixed">
+      <parent link="base_footprint"/>
+      <child link="base_link"/>
+      <origin xyz="0 0 ${wheel_radius}" rpy="0 0 0"/>
+    </joint>
+  </xacro:if>
   <link name="chassis_link">
     <inertial>
@@ -184,5 +194,5 @@
     <parent link="front_left_steering_link"/>
     <child link="front_left_wheel_link"/>
-    <origin xyz="0 ${(wheel_track - kingpin_width) / 2.0} 0" rpy="0 0 0"/>
+    <origin xyz="0 ${(front_wheel_track - kingpin_width) / 2.0} 0" rpy="0 0 0"/>
     <axis xyz="0 1 0"/>
     <limit effort="30" velocity="30"/>
@@ -192,5 +202,5 @@
     <parent link="front_right_steering_link"/>
     <child link="front_right_wheel_link"/>
-    <origin xyz="0 ${-(wheel_track - kingpin_width) / 2.0} 0" rpy="0 0 0"/>
+    <origin xyz="0 ${-(front_wheel_track - kingpin_width) / 2.0} 0" rpy="0 0 0"/>
     <axis xyz="0 1 0"/>
     <limit effort="30" velocity="30"/>
@@ -200,5 +210,5 @@
     <parent link="base_link"/>
     <child link="rear_left_wheel_link"/>
-    <origin xyz="${rear_axle_x} ${wheel_track / 2.0} 0" rpy="0 0 0"/>
+    <origin xyz="${rear_axle_x} ${rear_wheel_track / 2.0} 0" rpy="0 0 0"/>
     <axis xyz="0 1 0"/>
     <limit effort="50" velocity="30"/>
@@ -208,5 +218,5 @@
     <parent link="base_link"/>
     <child link="rear_right_wheel_link"/>
-    <origin xyz="${rear_axle_x} ${-wheel_track / 2.0} 0" rpy="0 0 0"/>
+    <origin xyz="${rear_axle_x} ${-rear_wheel_track / 2.0} 0" rpy="0 0 0"/>
     <axis xyz="0 1 0"/>
     <limit effort="50" velocity="30"/>
@@ -229,8 +239,7 @@
     <parent link="base_link"/>
     <child link="laser_link"/>
-    <origin xyz="${front_laser_x} 0 ${laser_z_from_ground - wheel_radius}" rpy="0 0 0"/>
-  </joint>
-  <!-- Rear sensor is physically symmetric about the vehicle geometric centre,
-       which is intentionally not the base_link origin. -->
+    <origin xyz="${front_laser_x} 0 ${front_laser_z}" rpy="0 0 0"/>
+  </joint>
+  <!-- Rear scan frame preserves the measured asymmetric installation. -->
   <link name="rear_laser_link">
     <inertial>
@@ -249,7 +258,9 @@
     <parent link="base_link"/>
     <child link="rear_laser_link"/>
-    <origin xyz="${rear_laser_x} 0 ${laser_z_from_ground - wheel_radius}"
+    <origin xyz="${rear_laser_x} 0 ${rear_laser_z}"
             rpy="0 0 ${pi}"/>
   </joint>
-  <xacro:include filename="turtle_car.gazebo.xacro"/>
+  <xacro:if value="$(arg include_gazebo)">
+    <xacro:include filename="turtle_car.gazebo.xacro"/>
+  </xacro:if>
 </robot>
